File: KiCad "original" PCB/SD_interrupter/SD_interrupter.kicad_pcb (KiCad board)
At the start: 2 copper layers, 83.8 x 86.4 mm, 39 parts, among them J1 Micro_SD_Card_Det, J2 AVR-ISP-6, J3 DIN-5, J4 Jack-DC, J5 VCC, SW1 BL_SW, SW2 MAIN_SW, SW3 UP_SW, SW4 DN_SW, SW5 OK_SW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

Commit message: 5V regulator footprint change
Parts:
- C1, C2, C3: value 1uF -> 47uF; footprint Capacitor_THT:C_Disc_D5.1mm_W3.2mm_P5.00mm -> Capacitor_THT:CP_Radial_D4.0mm_P1.50mm
- U1: value LM7805_TO220 -> AZ1117-5.0; footprint Package_TO_SOT_THT:TO-220-3_Vertical -> Package_TO_SOT_SMD:SOT-223-3_TabPin2
- moved U1 33.9 mm to (32.8, 56.1), turned to 90 degrees
- moved C2 23.9 mm to (36.1, 47.2)
- moved C3 11.1 mm to (40.9, 47.2), turned to 0 degrees
- moved C1 8.30 mm to (31.2, 47.2)
- moved U3 8.07 mm to (40.6, 56.1)
- moved C7 4.95 mm to (59.7, 50.3)
Connections:
- U1 pad 1: Net-(C1-Pad1) -> GND
- U1 pad 2: GND -> +5V
- U1 pad 3: +5V -> Net-(C1-Pad1)
Routing:
- net Net-(C1-Pad1): track 51.2 -> 23.3 mm, vias 0 -> 1
- net +3.3V: track 64.6 -> 78.6 mm, vias 1 -> 0
- net +5V: track 246.2 -> 258.8 mm
