File: KiCad "original" PCB/SD_interrupter/SD_interrupter.kicad_sch (KiCad schematic)
At the start: 39 parts, among them J1 Micro_SD_Card_Det, J2 AVR-ISP-6, J3 DIN-5, J4 Jack-DC, J5 VCC, SW1 BL_SW, SW2 MAIN_SW, SW3 UP_SW, SW4 DN_SW, SW5 OK_SW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

Commit message: 5V regulator footprint change
Parts:
- removed U1: LM7805_TO220, Package_TO_SOT_THT:TO-220-3_Vertical, symbol Regulator_Linear:LM7805_TO220
- added U1: AZ1117-5.0, Package_TO_SOT_SMD:SOT-223-3_TabPin2, symbol Regulator_Linear:AZ1117-5.0
- C1, C2, C3: value 1uF -> 47uF; footprint Capacitor_THT:C_Disc_D5.1mm_W3.2mm_P5.00mm -> Capacitor_THT:CP_Radial_D4.0mm_P1.50mm
Connections:
- net +5V: now also U1.2 (VO)
- net GND: now also U1.1 (GND)
- net at C1.1, SW2.1 (A): now also U1.3 (VI)
Changed lines of the file:
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@@
       (effects (font (size 1.27 1.27)) (justify left))
     )
-    (property "Value" "1uF" (id 1) (at 127 162.56 0)
-      (effects (font (size 1.27 1.27)) (justify left))
-    )
-    (property "Footprint" "Capacitor_THT:C_Disc_D5.1mm_W3.2mm_P5.00mm" (id 2) (at 124.1552 165.1 0)
+    (property "Value" "47uF" (id 1) (at 127 162.56 0)
+      (effects (font (size 1.27 1.27)) (justify left))
+    )
+    (property "Footprint" "Capacitor_THT:CP_Radial_D4.0mm_P1.50mm" (id 2) (at 124.1552 165.1 0)
       (effects (font (size 1.27 1.27)) hide)
     )
@@
     )
     (pin "1")
+  )
+  (symbol (lib_id "Regulator_Linear:AZ1117-5.0") (at 82.55 152.4 0) (unit 1)
+    (in_bom yes) (on_board yes) (fields_autoplaced)
+    (property "Reference" "U1" (id 0) (at 82.55 144.78 0))
+    (property "Value" "AZ1117-5.0" (id 1) (at 82.55 147.32 0))
+    (property "Footprint" "Package_TO_SOT_SMD:SOT-223-3_TabPin2" (id 2) (at 82.55 146.05 0)
+      (effects (font (size 1.27 1.27) italic) hide)
+    )
+    (property "Datasheet" "https://www.diodes.com/assets/Datasheets/AZ1117.pdf" (id 3) (at 82.55 152.4 0)
+      (effects (font (size 1.27 1.27)) hide)
+    )
+    (pin "1")
+    (pin "2")
+    (pin "3")
   )
   (symbol (lib_id "BH123A:BH123A") (at 154.94 160.02 270) (unit 1)
@@
       (effects (font (size 1.27 1.27)) (justify left))
     )
-    (property "Value" "1uF" (id 1) (at 73.66 162.56 0)
-      (effects (font (size 1.27 1.27)) (justify left))
-    )
-    (property "Footprint" "Capacitor_THT:C_Disc_D5.1mm_W3.2mm_P5.00mm" (id 2) (at 70.8152 165.1 0)
+    (property "Value" "47uF" (id 1) (at 73.66 162.56 0)
+      (effects (font (size 1.27 1.27)) (justify left))
+    )
+    (property "Footprint" "Capacitor_THT:CP_Radial_D4.0mm_P1.50mm" (id 2) (at 70.8152 165.1 0)
       (effects (font (size 1.27 1.27)) hide)
     )
@@
       (effects (font (size 1.27 1.27)) (justify left))
     )
-    (property "Value" "1uF" (id 1) (at 99.06 162.56 0)
-      (effects (font (size 1.27 1.27)) (justify left))
-    )
-    (property "Footprint" "Capacitor_THT:C_Disc_D5.1mm_W3.2mm_P5.00mm" (id 2) (at 96.2152 165.1 0)
+    (property "Value" "47uF" (id 1) (at 99.06 162.56 0)
+      (effects (font (size 1.27 1.27)) (justify left))
+    )
+    (property "Footprint" "Capacitor_THT:CP_Radial_D4.0mm_P1.50mm" (id 2) (at 96.2152 165.1 0)
       (effects (font (size 1.27 1.27)) hide)
     )
@@
     (pin "5")
   )
-  (symbol (lib_id "Regulator_Linear:LM7805_TO220") (at 82.55 152.4 0) (unit 1)
-    (in_bom yes) (on_board yes) (fields_autoplaced)
-    (property "Reference" "U1" (id 0) (at 82.55 144.78 0))
-    (property "Value" "LM7805_TO220" (id 1) (at 82.55 147.32 0))
-    (property "Footprint" "Package_TO_SOT_THT:TO-220-3_Vertical" (id 2) (at 82.55 146.685 0)
-      (effects (font (size 1.27 1.27) italic) hide)
-    )
-    (property "Datasheet" "https://www.onsemi.cn/PowerSolutions/document/MC7800-D.PDF" (id 3) (at 82.55 153.67 0)
-      (effects (font (size 1.27 1.27)) hide)
-    )
-    (pin "1")
-    (pin "2")
-    (pin "3")
-  )
   (symbol (lib_id "Device:R") (at 265.43 134.62 180) (unit 1)
     (in_bom yes) (on_board yes) (fields_autoplaced)
@@
     )
     (path "/85109c4c-57fe-41f9-b17f-9da0a29a4202"
-      (reference "C1") (unit 1) (value "1uF") (footprint "Capacitor_THT:C_Disc_D5.1mm_W3.2mm_P5.00mm")
+      (reference "C1") (unit 1) (value "47uF") (footprint "Capacitor_THT:CP_Radial_D4.0mm_P1.50mm")
     )
     (path "/8dbe64b9-086a-4695-a9a8-446d635d187c"
-      (reference "C2") (unit 1) (value "1uF") (footprint "Capacitor_THT:C_Disc_D5.1mm_W3.2mm_P5.00mm")
+      (reference "C2") (unit 1) (value "47uF") (footprint "Capacitor_THT:CP_Radial_D4.0mm_P1.50mm")
     )
     (path "/21982487-e555-47a1-a3a8-2147f30a76bc"
-      (reference "C3") (unit 1) (value "1uF") (footprint "Capacitor_THT:C_Disc_D5.1mm_W3.2mm_P5.00mm")
+      (reference "C3") (unit 1) (value "47uF") (footprint "Capacitor_THT:CP_Radial_D4.0mm_P1.50mm")
     )
     (path "/4402c666-7c01-421e-a26e-0ab99ddb36a3"
@@
       (reference "SW6") (unit 1) (value "BL_SW") (footprint "Switch:Switch 12x6mm")
     )
-    (path "/fa495c25-f5e1-4425-ae98-e5a137fd7f85"
-      (reference "U1") (unit 1) (value "LM7805_TO220") (footprint "Package_TO_SOT_THT:TO-220-3_Vertical")
+    (path "/2fec871f-a914-4c57-97ff-e1b1db97feb6"
+      (reference "U1") (unit 1) (value "AZ1117-5.0") (footprint "Package_TO_SOT_SMD:SOT-223-3_TabPin2")
     )
     (path "/e0db26c6-512a-4890-af7c-c5bad17096e1"
